File: Kicad/Guidon_v1a/Guidon_v1a.sch (KiCad schematic (older format))
At the start: 0 parts

Commit message: Update Schematic
Parts:
- added C1: 10u, symbol Device:CP1
- added C10, C11, C12, C5, C6, C7, C8, C9: 680n, symbol Device:C
- added C2: 100u, symbol Device:CP1
- added C3, C4: 100n, symbol Device:C
- added D1: D_Schottky_AKA, symbol Device:D_Schottky_AKA
- added IC1: R-785.0-0.5, RECOM_R-785.0-0.5, symbol R-785.0-0.5:R-785.0-0.5
- added IC2: MCP2562, Package_SO:SOIC-8_3.9x4.9mm_P1.27mm, symbol Interface_CAN_LIN:MCP2562-E-SN
- added K1: ALIM, symbol Connector_Generic:Conn_01x02
- added K2: BUS CAN, symbol Connector_Generic:Conn_01x02
- added K3: INTER., symbol Connector_Generic:Conn_01x09
- added K4: OLED, symbol Connector_Generic:Conn_01x04
- added R1: 120, symbol Device:R
- added R10, R2, R3, R4, R5, R6, R7, R8: 6.8k, symbol Device:R
- added R11, R9: 3.3k, symbol Device:R
- added UC1: BluePill STM32, symbol YAAJ_STM32:BluePill_1
Connections:
- new net: IC2.6 (CANL), K2.2 (Pin_2), R1.2
- new net: IC2.7 (CANH), K2.1 (Pin_1), R1.1
- new net: C1.1, D1.2 (K), IC1.1 (+VIN)
- new net: D1.1 (A), D1.3 (A), K1.1 (Pin_1)
- new net +5V: C2.1, C4.2, IC1.3 (+VOUT), IC2.3 (VDD), UC1.18 (5V)
- new net BP0: C5.1, K3.1 (Pin_1), R2.2, UC1.25 (PA0)
- new net BP1: C6.1, K3.2 (Pin_2), R3.2, UC1.26 (PA1)
- new net BP2: C7.1, K3.3 (Pin_3), R4.2, UC1.27 (PA2)
- new net BP3: C8.1, K3.4 (Pin_4), R5.2, UC1.28 (PA3)
- new net BP4: C9.1, K3.5 (Pin_5), R6.2, UC1.29 (PA4)
- new net BP5: C10.1, K3.6 (Pin_6), R7.2, UC1.30 (PA5)
- new net BP6: C11.1, K3.7 (Pin_7), R8.2, UC1.31 (PA6)
- new net BP7: C12.1, K3.8 (Pin_8), R10.2, UC1.32 (PA7)
- new net CANRX: IC2.4 (RXD), UC1.8 (PA11)
- new net CANTX: IC2.1 (TXD), UC1.9 (PA12)
- new net GND: C1.2, C10.2, C11.2, C12.2, C2.2, C3.2, C4.1, C5.2, C6.2, C7.2, C8.2, C9.2, IC1.2 (GND), IC2.2 (VSS), IC2.8 (STBY), K1.2 (Pin_2), K3.9 (Pin_9), K4.2 (Pin_2), UC1.19 (GND), UC1.39 (GND), UC1.40 (GND)
- new net SCL: K4.3 (Pin_3), R11.2, UC1.14 (PB6)
- new net SDA: K4.4 (Pin_4), R9.2, UC1.15 (PB7)
- new net VCC: C3.1, IC2.5 (Vio), K4.1 (Pin_1), R10.1, R11.1, R2.1, R3.1, R4.1, R5.1, R6.1, R7.1, R8.1, R9.1, UC1.20 (3V3)
- no-connect marks 0 -> 23

Commit message: Update projet
Parts:
- D1: value D_Schottky_AKA -> MBRD340
- R11, R9: value 3.3k -> 4.7k
- renumbered C3 to C1, C1 to C2, C4 to C3, C2 to C4, IC2 to IC1, IC1 to IC2
Other:
- moved on the sheet: C1, C10, C11, C12, C2, C3, C4, C5, C6, C7, C8, C9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

Commit message: Update
Other:
- note added: "*"
- moved on the sheet: R11, R9
Changed lines of the file:
@@
 Wire Wire Line
 	7200 2400 9200 2400
-Connection ~ 9600 4600
-Wire Wire Line
-	9600 4400 9600 4600
+Connection ~ 9400 4600
+Wire Wire Line
+	9400 4400 9400 4600
 $Comp
 L power:VCC #PWR018
 U 1 1 5E95D1B8
-P 9600 4400
-F 0 "#PWR018" H 9600 4250 50  0001 C CNN
-F 1 "VCC" H 9617 4573 50  0000 C CNN
-F 2 "" H 9600 4400 50  0001 C CNN
-F 3 "" H 9600 4400 50  0001 C CNN
-	1    9600 4400
-	1    0    0    -1
-$EndComp
-Wire Wire Line
-	9600 4600 9600 4800
-Wire Wire Line
-	9300 4600 9600 4600
-Wire Wire Line
-	9300 4800 9300 4600
+P 9400 4400
+F 0 "#PWR018" H 9400 4250 50  0001 C CNN
+F 1 "VCC" H 9417 4573 50  0000 C CNN
+F 2 "" H 9400 4400 50  0001 C CNN
+F 3 "" H 9400 4400 50  0001 C CNN
+	1    9400 4400
+	1    0    0    -1
+$EndComp
+Wire Wire Line
+	9400 4600 9400 4800
+Wire Wire Line
+	9100 4600 9400 4600
+Wire Wire Line
+	9100 4800 9100 4600
 Text GLabel 7200 2500 0    50   Output ~ 0
 BP7
@@
 Wire Wire Line
 	7400 1700 7400 1800
-Text GLabel 9100 5300 0    50   BiDi ~ 0
+Text GLabel 8900 5300 0    50   BiDi ~ 0
 SDA
-Text GLabel 9100 5200 0    50   Input ~ 0
+Text GLabel 8900 5200 0    50   Input ~ 0
 SCL
-Connection ~ 9600 5200
-Wire Wire Line
-	9600 5200 9100 5200
-Connection ~ 9300 5300
-Wire Wire Line
-	9300 5300 9100 5300
-Wire Wire Line
-	9300 5300 9300 5100
-Wire Wire Line
-	10000 5300 9300 5300
-Wire Wire Line
-	9600 5200 9600 5100
-Wire Wire Line
-	10000 5200 9600 5200
-$Comp
-L Device:R R9
-U 1 1 5E8F55B0
-P 9300 4950
-F 0 "R9" H 9370 4996 50  0000 L CNN
-F 1 "4.7k" H 9370 4905 50  0000 L CNN
-F 2 "" V 9230 4950 50  0001 C CNN
-F 3 "~" H 9300 4950 50  0001 C CNN
-	1    9300 4950
-	1    0    0    -1
-$EndComp
+Wire Wire Line
+	9400 5200 8900 5200
+Wire Wire Line
+	9100 5300 8900 5300
+Wire Wire Line
+	9100 5300 9100 5100
+Wire Wire Line
+	9400 5200 9400 5100
 $Comp
 L Device:R R11
 U 1 1 5E8F474D
-P 9600 4950
-F 0 "R11" H 9670 4996 50  0000 L CNN
-F 1 "4.7k" H 9670 4905 50  0000 L CNN
-F 2 "" V 9530 4950 50  0001 C CNN
-F 3 "~" H 9600 4950 50  0001 C CNN
-	1    9600 4950
+P 9400 4950
+F 0 "R11" H 9470 4996 50  0000 L CNN
+F 1 "4.7k" H 9470 4905 50  0000 L CNN
+F 2 "" V 9330 4950 50  0001 C CNN
+F 3 "~" H 9400 4950 50  0001 C CNN
+	1    9400 4950
 	1    0    0    -1
 $EndComp
@@
 $EndComp
 NoConn ~ 3150 1400
+$Comp
+L Device:R R9
+U 1 1 5E8F55B0
+P 9100 4950
+F 0 "R9" H 9170 4996 50  0000 L CNN
+F 1 "4.7k" H 9170 4905 50  0000 L CNN
+F 2 "" V 9030 4950 50  0001 C CNN
+F 3 "~" H 9100 4950 50  0001 C CNN
+	1    9100 4950
+	1    0    0    -1
+$EndComp
+Wire Wire Line
+	10000 5200 9400 5200
+Connection ~ 9400 5200
+Wire Wire Line
+	10000 5300 9100 5300
+Connection ~ 9100 5300
+Wire Notes Line
+	9000 4750 9700 4750
+Wire Notes Line
+	9700 4750 9700 5150
+Wire Notes Line
+	9700 5150 9000 5150
+Wire Notes Line
+	9000 5150 9000 4750
+Text Notes 9600 5150 0    50   ~ 0
+*
 $EndSCHEMATC

Commit message: Update schema
Parts:
- removed R11, R9: 4.7k, symbol Device:R
- renumbered R10 to R9
Other:
- note removed: "*"
Changed lines of the file:
@@
 Wire Wire Line
 	7200 2400 9200 2400
-Connection ~ 9400 4600
-Wire Wire Line
-	9400 4400 9400 4600
-$Comp
-L power:VCC #PWR018
-U 1 1 5E95D1B8
-P 9400 4400
-F 0 "#PWR018" H 9400 4250 50  0001 C CNN
-F 1 "VCC" H 9417 4573 50  0000 C CNN
-F 2 "" H 9400 4400 50  0001 C CNN
-F 3 "" H 9400 4400 50  0001 C CNN
-	1    9400 4400
-	1    0    0    -1
-$EndComp
-Wire Wire Line
-	9400 4600 9400 4800
-Wire Wire Line
-	9100 4600 9400 4600
-Wire Wire Line
-	9100 4800 9100 4600
 Text GLabel 7200 2500 0    50   Output ~ 0
 BP7
@@
 Wire Wire Line
 	7400 1700 7400 1800
-Text GLabel 8900 5300 0    50   BiDi ~ 0
+Text GLabel 9800 5300 0    50   BiDi ~ 0
 SDA
-Text GLabel 8900 5200 0    50   Input ~ 0
+Text GLabel 9800 5200 0    50   Input ~ 0
 SCL
 Wire Wire Line
-	9400 5200 8900 5200
-Wire Wire Line
-	9100 5300 8900 5300
-Wire Wire Line
-	9100 5300 9100 5100
-Wire Wire Line
-	9400 5200 9400 5100
-$Comp
-L Device:R R11
-U 1 1 5E8F474D
-P 9400 4950
-F 0 "R11" H 9470 4996 50  0000 L CNN
-F 1 "4.7k" H 9470 4905 50  0000 L CNN
-F 2 "" V 9330 4950 50  0001 C CNN
-F 3 "~" H 9400 4950 50  0001 C CNN
-	1    9400 4950
-	1    0    0    -1
-$EndComp
-Wire Wire Line
 	9900 5100 9900 5400
 Wire Wire Line
 	10000 5100 9900 5100
 $Comp
-L power:GND #PWR020
+L power:GND #PWR019
 U 1 1 5E8ECFA8
 P 9900 5400
-F 0 "#PWR020" H 9900 5150 50  0001 C CNN
+F 0 "#PWR019" H 9900 5150 50  0001 C CNN
 F 1 "GND" H 9905 5227 50  0000 C CNN
 F 2 "" H 9900 5400 50  0001 C CNN
@@
 	10000 5000 9900 5000
 $Comp
-L power:VCC #PWR019
+L power:VCC #PWR018
 U 1 1 5E8EA57B
 P 9900 4900
-F 0 "#PWR019" H 9900 4750 50  0001 C CNN
+F 0 "#PWR018" H 9900 4750 50  0001 C CNN
 F 1 "VCC" H 9917 5073 50  0000 C CNN
 F 2 "" H 9900 4900 50  0001 C CNN
@@
 $EndComp
 $Comp
-L Device:R R10
+L Device:R R9
 U 1 1 5E8552AB
 P 9500 1550
-F 0 "R10" H 9570 1596 50  0000 L CNN
+F 0 "R9" H 9570 1596 50  0000 L CNN
 F 1 "6.8k" H 9570 1505 50  0000 L CNN
 F 2 "" V 9430 1550 50  0001 C CNN
@@
 $EndComp
 NoConn ~ 3150 1400
-$Comp
-L Device:R R9
-U 1 1 5E8F55B0
-P 9100 4950
-F 0 "R9" H 9170 4996 50  0000 L CNN
-F 1 "4.7k" H 9170 4905 50  0000 L CNN
-F 2 "" V 9030 4950 50  0001 C CNN
-F 3 "~" H 9100 4950 50  0001 C CNN
-	1    9100 4950
-	1    0    0    -1
-$EndComp
-Wire Wire Line
-	10000 5200 9400 5200
-Connection ~ 9400 5200
-Wire Wire Line
-	10000 5300 9100 5300
-Connection ~ 9100 5300
-Wire Notes Line
-	9000 4750 9700 4750
-Wire Notes Line
-	9700 4750 9700 5150
-Wire Notes Line
-	9700 5150 9000 5150
-Wire Notes Line
-	9000 5150 9000 4750
-Text Notes 9600 5150 0    50   ~ 0
-*
+Wire Wire Line
+	9800 5200 10000 5200
+Wire Wire Line
+	9800 5300 10000 5300
 $EndSCHEMATC

Commit message: Update
Parts:
- removed C10, C11, C12, C9: 680n, symbol Device:C
- removed C2: 10u, symbol Device:CP1
- removed IC2: R-785.0-0.5, RECOM_R-785.0-0.5, symbol R-785.0-0.5:R-785.0-0.5
- removed K1: ALIM, symbol Connector_Generic:Conn_01x02
- removed K3: INTER., symbol Connector_Generic:Conn_01x09
- removed R7, R8, R9: 6.8k, symbol Device:R
- removed UC1: BluePill STM32, symbol YAAJ_STM32:BluePill_1
- added C1, C2: 22p, symbol Device:C
- added C10, C11, C12, C3, C6, C7, C9: 10u, symbol Device:CP1
- added C13, C14, C19, C20, C21, C22, C23, C24, C25, C26, C27: 680n, symbol Device:C
- added IC2: L7805CDT, symbol Regulator_Linear:L7805
- added IC3: DSPIC30F4012, SOIC127P1030X265-28N, symbol DSPIC30F4012-20I_SO:DSPIC30F4012-20I_SO
- added IC4: AMS1117-3.3, symbol Regulator_Linear:LM1117-3.3
- added K1: ICSP, symbol Connector_Generic:Conn_01x06
- added K2: ALIM, symbol Connector_Generic:Conn_01x02
- added K4: BP OLED, symbol Connector_Generic:Conn_01x03
- added K6: GUIDON G, symbol Connector_Generic:Conn_01x05
- added K7: FREIN, symbol Connector_Generic:Conn_01x02
- added K8: GUIDON D, symbol Connector_Generic:Conn_01x05
- added K9: RESERVE, symbol Connector_Generic:Conn_01x05
- added R1: 10k, symbol Device:R
- added R11, R12, R13, R14, R15, R16, R17, R18, R19, R5: 6.8k, symbol Device:R
- added R2, R3: 1.8k, symbol Device:R
- added X1: 8M, symbol Device:Crystal
- C4: value 100u -> 10u
- D1: value MBRD340 -> VS-MBRD340
- K5: renamed from K4; value OLED -> AFF OLED
- renumbered C5 to C15, C6 to C16, C7 to C17, C8 to C18, C1 to C5, C3 to C8, K2 to K3, R5 to R10, R1 to R4, R2 to R7, R3 to R8, R4 to R9
Connections:
- net +5V: now also C10.1, C9.1, IC2.3 (OUT), IC4.3 (VI); no longer C4.1
- net GND: now also C1.2, C10.2, C11.2, C12.2, C13.2, C14.2, C19.2, C2.2, C20.2, C21.2, C22.2, C23.2, C24.2, C25.2, C26.2, C27.2, C3.2, C6.2, C7.2, C9.2, IC2.2 (GND), IC3.19 (VSS), IC3.27 (AVSS), IC3.8 (VSS_2), IC4.1 (GND), K1.3 (Pin_3), K2.2 (Pin_2), K4.3 (Pin_3), K6.5 (Pin_5), K7.2 (Pin_2), K8.5 (Pin_5), K9.5 (Pin_5)
- net SCL: now also IC3.14 (EMUD2/OC2/IC2/INT2/RD1)
- net SDA: now also IC3.15 (EMUC2/OC1/IC1/INT1/RD0)
- net VCC: now also C11.1, C12.1, IC3.13 (VDD_2), IC3.20 (VDD), IC3.28 (AVDD), IC4.2 (VO), K1.2 (Pin_2), R1.1, R11.1, R12.1, R13.1, R14.1, R15.1, R16.1, R17.1, R18.1, R19.1, R5.1
- net at D1.2 (K): now also C4.1, C3.1, C6.1, C7.1, IC2.1 (IN)
- net at D1.1 (A), D1.3 (A): now also K2.1 (Pin_1)
- net BP0 renamed BPG0
- net BPG0: now also IC3.2 (EMUD3/AN0/VREF+/CN2/RB0), K6.1 (Pin_1)
- net BP1 renamed BPG1
- net BPG1: now also IC3.3 (EMUC3/AN1/VREF-/CN3/RB1), K6.2 (Pin_2)
- net BP2 renamed BPG2
- net BPG2: now also IC3.4 (AN2/~SS1~/CN4/RB2), K6.3 (Pin_3)
- net BP3 renamed BPG3
- net BPG3: now also IC3.5 (AN3/INDX/CN5/RB3), K6.4 (Pin_4)
- net BP4 renamed BPA1
- net BPA1: now also C14.1, IC3.16 (FLTA/INT0/SCK1/OCFA/RE8), K4.2 (Pin_2)
- net CANRX: no longer names the net of IC1.4 (RXD)
- net CANRX: now also R3.1
- net CANTX: no longer names the net of IC1.1 (TXD)
- net CANTX: now also R2.1
- new net: C2.1, IC3.9 (OSC1/CLKI), X1.2
- new net BPA0: C13.1, IC3.21 (PWM3H/RE5), K4.1 (Pin_1), R5.2
- new net BPD0: C20.1, IC3.26 (PWM1L/RE0), K8.1 (Pin_1), R12.2
- new net BPD1: C22.1, IC3.25 (PWM1H/RE1), K8.2 (Pin_2), R14.2
- new net BPD2: C24.1, IC3.24 (PWM2L/RE2), K8.3 (Pin_3), R16.2
- new net BPD3: C26.1, IC3.23 (PWM2H/RE3), K8.4 (Pin_4), R18.2
- new net FREIN: C19.1, IC3.22 (PWM3L/RE4), K7.1 (Pin_1), R11.2
- new net OSC2: C1.1, IC3.10 (OSC2/CLKO/RC15), X1.1
- new net PGC: IC3.18 (PGC/EMUC/U1RX/SDI1/SDA/C1RX/RF2), K1.5 (Pin_5), R3.2
- new net PGD: IC3.17 (PGD/EMUD/U1TX/SDO1/SCL/C1TX/RF3), K1.4 (Pin_4), R2.2
- new net RES0: C21.1, IC3.6 (AN4/QEA/IC7/CN6/RB4), K9.1 (Pin_1), R13.2
- new net RES1: C23.1, IC3.7 (AN5/QEB/IC8/CN7/RB5), K9.2 (Pin_2), R15.2
- new net RES2: C25.1, IC3.11 (EMUD1/SOSCI/T2CK/U1ATX/CN1/RC13), K9.3 (Pin_3), R17.2
- new net RES3: C27.1, IC3.12 (EMUC1/SOSCO/T1CK/U1ARX/CN0/RC14), K9.4 (Pin_4), R19.2
- new net ~MCLR: IC3.1 (~MCLR), K1.1 (Pin_1), R1.2
- no-connect marks 23 -> 1
Other:
- moved on the sheet: C15, C16, C17, C18, C5, C8, IC1, K3, K5, R10, R4, R7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

Commit message: Update
Parts:
- removed C13, C14, C19, C20, C21, C22, C23, C24, C25, C26, C27: 680n, symbol Device:C
- removed R11, R12, R13, R14, R15, R16, R17, R18, R19, R5, R6: 6.8k, symbol Device:R
Connections:
- net GND: no longer K4.3 (Pin_3), K6.5 (Pin_5), K7.2 (Pin_2), K8.5 (Pin_5), K9.5 (Pin_5)
- net RES2: no longer K9.3 (Pin_3)
- net RES3: no longer K9.4 (Pin_4)
- net BPA0: no longer names the net of IC3.21 (PWM3H/RE5)
- net BPA0: no longer K4.1 (Pin_1)
- net BPA1: no longer names the net of IC3.16 (FLTA/INT0/SCK1/OCFA/RE8)
- net BPA1: no longer K4.2 (Pin_2)
- net BPD0 renamed BPL0
- net BPL0: now also C15.1, K6.1 (Pin_1), K7.1 (Pin_1), K9.1 (Pin_1), R7.2
- net BPD1 renamed BPL1
- net BPL1: now also C16.1, K4.1 (Pin_1), K6.2 (Pin_2), K9.2 (Pin_2), R8.2
- net BPD2 renamed BPL2
- net BPL2: now also C17.1, K4.2 (Pin_2), K6.3 (Pin_3), K9.3 (Pin_3), R9.2
- net BPD3 renamed BPL3
- net BPL3: now also C18.1, K6.4 (Pin_4), K9.4 (Pin_4), R10.2
- removed net BPG0: C15.1, IC3.2 (EMUD3/AN0/VREF+/CN2/RB0), K6.1 (Pin_1), R7.2
- removed net BPG1: C16.1, IC3.3 (EMUC3/AN1/VREF-/CN3/RB1), K6.2 (Pin_2), R8.2
- removed net BPG2: C17.1, IC3.4 (AN2/~SS1~/CN4/RB2), K6.3 (Pin_3), R9.2
- removed net BPG3: C18.1, IC3.5 (AN3/INDX/CN5/RB3), K6.4 (Pin_4), R10.2
- net FREIN: no longer names the net of IC3.22 (PWM3L/RE4)
- net FREIN: no longer K7.1 (Pin_1)
- net RES0: no longer names the net of IC3.6 (AN4/QEA/IC7/CN6/RB4)
- net RES0: no longer K9.1 (Pin_1)
- net RES1: no longer names the net of IC3.7 (AN5/QEB/IC8/CN7/RB5)
- net RES1: no longer K9.2 (Pin_2)
- new net BPDIV: IC3.5 (AN3/INDX/CN5/RB3), K4.3 (Pin_3), K7.2 (Pin_2)
- new net BPGD: IC3.3 (EMUC3/AN1/VREF-/CN3/RB1), K8.5 (Pin_5)
- new net BPGG: IC3.2 (EMUD3/AN0/VREF+/CN2/RB0), K6.5 (Pin_5)
- new net BPRES: IC3.4 (AN2/~SS1~/CN4/RB2), K9.5 (Pin_5)
- no-connect marks 1 -> 6
Other:
- moved on the sheet: C15, C16, C17, C18, C5, C8, IC1, K3, K4, K5, K6, K7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

Commit message: Update
Parts:
- added C? (x3): 100n, symbol Device:C
- renumbered C15 to C?, C16 to C?, C17 to C?, C18 to C?, C1 to C?, C2 to C?, C8 to C?, C5 to C?, C9 to C?, C10 to C?, C11 to C?, C12 to C?, C3 to C?, C4 to C?, C6 to C?, C7 to C?, D1 to D?, IC1 to IC?, IC4 to IC?, IC3 to IC?, IC2 to IC?, K6 to K?, K5 to K?, K8 to K?, K2 to K?, K3 to K?, K4 to K?, K9 to K?, K1 to K?, K7 to K?, R7 to R?, R8 to R?, R9 to R?, R10 to R?, R4 to R?, R2 to R?, R3 to R?, R1 to R?, X1 to X?
Connections:
- net BPDIV: now also IC?.3 (EMUC3/AN1/VREF-/CN3/RB1); no longer IC?.5 (AN3/INDX/CN5/RB3)
- net BPGD: now also IC?.4 (AN2/~SS1~/CN4/RB2); no longer IC?.3 (EMUC3/AN1/VREF-/CN3/RB1)
- net BPRES: now also IC?.5 (AN3/INDX/CN5/RB3); no longer IC?.4 (AN2/~SS1~/CN4/RB2)
- net GND: now also C?.2, C?.2, C?.2
- net VCC: now also C?.1, C?.1, C?.1

Commit message: Update
Parts:
- gave numbers to parts that had none: 42
